Commit message: 导航配置成功 建图完成 待进行测试代码

File: src/sweeper_robot_omni4_base_ros/urdf/sweeper_robot_omni4_base.urdf (robot description, URDF)
Before this commit: robot sweeper_robot_omni4_base, 9 links, 8 joints
Links:
- removed link cmd_vel_interface_link
- removed link odometry_link
- link base_link: geometry collision cylinder length=0.0600 radius=0.2500; visual box size=0.052 0.034 0.060
Joints:
- removed joint cmd_vel_interface_joint
- removed joint odometry_joint
- joint lidar_joint: origin xyz=0.000 0.075 0.1610 rpy=0 0 0 -> xyz=0 0 0.1610 rpy=0 0 0
