Commit message: fix: stabilize differential chassis pitch

File: src/sweeper_robot_diff2_submit_ros/urdf/sweeper_robot_diff2_submit.urdf (robot description, URDF)
Before this commit: robot sweeper_robot_diff2_submit, 5 links, 4 joints
Links:
- added link front_passive_support_link, mass 0.0100; collision sphere radius=0.0250
- added link rear_passive_support_link, mass 0.0100; collision sphere radius=0.0250
Joints:
- added joint front_passive_support_joint: type fixed, parent base_link, child front_passive_support_link, origin xyz=0.1800 0 0.0250 rpy=0 0 0
- added joint rear_passive_support_joint: type fixed, parent base_link, child rear_passive_support_link, origin xyz=-0.1800 0 0.0250 rpy=0 0 0
